Commit message: fix: use body_without_cam.stl to remove Zivid from RViz visual

File: yumi_ros2/yumi_description/urdf/yumi.urdf (robot description, URDF)
Before this commit: robot yumi, 24 links, 23 joints
Links:
- link yumi_body: geometry collision mesh filename=package://yumi_description/meshes/coarse/body.stl; visual mesh filename=package://yumi_description/meshes/body_without_cam.stl
